Commit message: new instruction task_manager: robotfault->tryagain (+new calibration camera comau)

File: urdf/bonmet/bonmetc60.urdf.xacro (robot description, xacro)
@@ -1,7 +1,8 @@
 <?xml version="1.0"?>
-<robot xmlns:sensor="http://playerstage.sourceforge.net/gazebo/xmlschema/#sensor" xmlns:controller="http://playerstage.sourceforge.net/gazebo/xmlschema/#controller"
-  xmlns:interface="http://playerstage.sourceforge.net/gazebo/xmlschema/#interface" xmlns:xacro="http://ros.org/wiki/xacro"
-  name="bonmetc60">
-<!--xacro:macro name="bonmetc60" params="prefix"-->
+<robot xmlns:sensor="http://playerstage.sourceforge.net/gazebo/xmlschema/#sensor"
+  xmlns:controller="http://playerstage.sourceforge.net/gazebo/xmlschema/#controller"
+  xmlns:interface="http://playerstage.sourceforge.net/gazebo/xmlschema/#interface"
+  xmlns:xacro="http://ros.org/wiki/xacro" name="bonmetc60">
+  <!--xacro:macro name="bonmetc60" params="prefix"-->
   <xacro:property name="robot_prefix" value="bonmetc60/" />
   <link name="${robot_prefix}base_link">
@@ -14,5 +15,5 @@
     <child link="${robot_prefix}link1" />
     <origin xyz="0.00 0 0.32" rpy="0 0 0" />
-    <limit effort="1000" velocity="1000" lower="-2.9670" upper="2.9670" /> <!-- TODO -->
+    <limit effort="1000" velocity="1000" lower="-2.9670" upper="2.9670" />
     <!-- -170,+170 -->
   </joint>
@@ -24,5 +25,5 @@
     <child link="${robot_prefix}link2" />
     <origin xyz="0.05 0 0.0" rpy="1.571 0 0" />
-    <limit effort="1000" velocity="1000" lower="-2.267" upper="1.57" />  <!-- TODO -->
+    <limit effort="1000" velocity="1000" lower="-2.267" upper="1.57" />
     <!-- -85,+155 -->
   </joint>
@@ -34,5 +35,5 @@
     <child link="${robot_prefix}link3" />
     <origin xyz="0 0.27 0" rpy="0 0 0" />
-    <limit effort="1000" velocity="1000" lower="-1.22" upper="1.483" />  <!-- TODO -->
+    <limit effort="1000" velocity="1000" lower="-1.22" upper="1.483" />
     <!-- -170,+0 -->
   </joint>
@@ -45,5 +46,5 @@
     <!-- <origin xyz="0.299 0.07 0.0" rpy="0 1.571 0" /> -->
     <origin xyz="0.299 0.07 0.0" rpy="0 1.571 0" />
-    <limit effort="1000" velocity="1000" lower="-2.967" upper="2.967" />  <!-- TODO -->
+    <limit effort="1000" velocity="1000" lower="-2.967" upper="2.967" />
   </joint>
   <link name="${robot_prefix}link5">
@@ -54,5 +55,5 @@
     <child link="${robot_prefix}link5" />
     <origin xyz="0.0 0.0 0.0" rpy="0.0 -1.57 0.0" />
-    <limit effort="1000" velocity="1000" lower="-1.74" upper="1.74" />  <!-- TODO -->
+    <limit effort="1000" velocity="1000" lower="-1.74" upper="1.74" />
     <!-- -130,+130 -->
   </joint>
@@ -64,16 +65,6 @@
     <child link="${robot_prefix}link6" />
     <origin xyz="0.0785 0 0.0" rpy="0 1.57 0" />
-    <limit effort="1000" velocity="1000" lower="-6.28" upper="6.28" />  <!-- TODO -->
+    <limit effort="1000" velocity="1000" lower="-6.28" upper="6.28" />
   </joint>
-  <!--
-  <link name="${robot_prefix}tool">
-  </link>
-  <joint name="${robot_prefix}link6_to_tool" type="continuous">
-    <axis xyz="0 0 1" />
-    <parent link="${robot_prefix}link6" />
-    <child link="${robot_prefix}tool" />
-    <origin xyz="0 0 -0.085" rpy="0 0 0" />
-  </joint>
--->
-<!--/xacro:macro-->
+  <!--/xacro:macro-->
 </robot>
